File: rpi_dual_rfm98_hat/rpi_dual_rfm98_hat.kicad_pcb (KiCad board)
At the start: 2 copper layers, 65 x 56 mm, 12 parts, among them J1 PJ-202A, P1 Conn_02x20_Odd_Even, SW1 SW_Push_Open_Dual, U1 E32400M30S, U2 OLED

Commit message: ready for review
Parts:
- removed SW1: SW_Push_Open_Dual, Button_Switch_SMD:SW_Push_1P1T_NO_6x6mm_H9.5mm
- added D1: LED, LED_SMD:LED_0603_1608Metric, F.Cu at (259.5, 127.3)
- added D2: LED, LED_SMD:LED_0603_1608Metric, F.Cu at (203.8, 116.6)
- added D3: LED, LED_SMD:LED_0603_1608Metric, F.Cu at (203.8, 138.6)
- added J2: Conn_Coaxial, Connector_Coaxial:SMA_Amphenol_132134-11_Vertical, F.Cu at (204.9, 107.9)
- added J3: Conn_Coaxial, Connector_Coaxial:SMA_Amphenol_132134-11_Vertical, F.Cu at (204.9, 129.8)
- added J4: Conn_01x03_Male, Connector_JST:JST_XH_B3B-XH-AM_1x03_P2.50mm_Vertical, F.Cu at (259.8, 109.7)
- J1: value PJ-202A -> Conn_01x02_Male; footprint PJ-202A:CUI_PJ-202A -> Connector_JST:JST_XH_B2B-XH-AM_1x02_P2.50mm_Vertical
- R1, R2: value 1k -> R_US; footprint Resistor_SMD:R_1206_3216Metric_Pad1.30x1.75mm_HandSolder -> Resistor_SMD:R_0603_1608Metric
- R3: value 10k -> R_US; footprint Resistor_SMD:R_1206_3216Metric_Pad1.30x1.75mm_HandSolder -> Resistor_SMD:R_0603_1608Metric
- U1: value E32400M30S -> RFM98PW-symbols; footprint TinyGS:E32400M -> mainboard:RFM95PW
- U2: value OLED -> RFM98PW-symbols; footprint TinyGS:OLED -> mainboard:RFM95PW
- moved R2 36.9 mm to (205.5, 116.6), turned to 90 degrees
- moved U2 33.7 mm to (229.2, 137.3), turned to 180 degrees
- moved U1 26.1 mm to (229.2, 115.4), turned to 180 degrees
- moved R3 20.3 mm to (205.5, 138.6), turned to 90 degrees
- moved R1 19.7 mm to (259.5, 125.6), turned to 180 degrees
- moved J1 14.6 mm to (259.8, 132.4)
Connections:
- P1 pad 1: +3V3 -> unconnected-(P1-Pad1)
- P1 pad 17: +3V3 -> unconnected-(P1-Pad17)
- R1 pad 1: Net-(R1-Pad1) -> Net-(D1-Pad1)
- R1 pad 2: /GPIO27(GEN2) -> GND
- R2 pad 1: Net-(R2-Pad1) -> Net-(D2-Pad1)
- R2 pad 2: /GPIO22(GEN3) -> GND
- R3 pad 1: +3V3 -> Net-(D3-Pad1)
- R3 pad 2: Net-(R3-Pad2) -> GND
- U1 pad 1: GND -> Net-(J2-Pad1)
- U1 pad 10: +5V -> /GPIO9(SPI0_MISO)
- U1 pad 11: GND -> /GPIO10(SPI0_MOSI)
- U1 pad 3: GND -> unconnected-(U1-Pad3)
- U1 pad 4: GND -> unconnected-(U1-Pad4)
- U1 pad 5: GND -> +5V
- U1 pad 6: Net-(R2-Pad1) -> /GPIO23(GEN4)
- U1 pad 7: Net-(R1-Pad1) -> unconnected-(U1-Pad7)
- U1 pad 9: +5V -> unconnected-(U1-Pad9)
- U2 pad 1: GND -> Net-(J3-Pad1)
- U2 pad 2: +3V3 -> GND
- U2 pad 3: /GPIO3(SCL1) -> unconnected-(U2-Pad3)
- U2 pad 4: /GPIO2(SDA1) -> unconnected-(U2-Pad4)
Routing:
- net /GPIO3(SCL1): track 148.0 -> 0.00 mm
- net /GPIO2(SDA1): track 146.4 -> 0.00 mm
- net +3V3: track 104.9 -> 0.00 mm
- net /GPIO17(GEN0): track 0.00 -> 61.0 mm, vias 0 -> 2
- net /GPIO5: track 59.2 -> 0.00 mm
- net /GPIO24(GEN5): track 0.00 -> 50.4 mm, vias 0 -> 1
- net /GPIO20(SPI1_MOSI): track 0.00 -> 48.5 mm, vias 0 -> 1
- net /GPIO21(SPI1_SCK): track 0.00 -> 48.1 mm, vias 0 -> 1
- net /GPIO19(SPI1_MISO): track 0.00 -> 46.4 mm, vias 0 -> 1
- net /GPIO8(SPI0_CE_N): track 0.00 -> 28.7 mm, vias 0 -> 1
- net /GPIO23(GEN4): track 55.8 -> 30.9 mm
- net /GPIO11(SPI0_SCK): track 50.4 -> 27.2 mm, vias 0 -> 2
- net /GPIO25(GEN6): track 45.9 -> 27.1 mm, vias 0 -> 1
- net /GPIO26: track 0.00 -> 15.8 mm
- net /GPIO27(GEN2): track 40.4 -> 27.7 mm
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Other:
- board text added: "+5V 3A"
- board text added: "GND"
- board text added: "RX/TX Switch"
- board text added: "TX RADIO - SPI0 CS: GPIO8 RESET: GPIO25 GPIO_0: GPIO23 TX LED: GPIO27 RX RADIO - SPI1 CS: GPIO21 RESET: GPIO24 GPIO_0: GPIO22 RX LED: GPIO17 RX/TX Switch: GPIO26"
